File: tinyusbboard.brd (EAGLE design)
At the start: 24.6 x 50 mm, 36 parts, among them IC1 MEGA8-AI, Q1 16MHz

Commit message: More conventional schematic and plus lower capacities to confirm to the USB maximum
Parts:
- C1A, C1B: value 1uF -> 100nF
- CAP: value 22uF -> 4.7uF
- D1, D2: value ZMM3V6 -> 3V6
- JP1: value (none) -> PDA
- JP2: value (none) -> PDB
- JP3: value (none) -> PDC
- JP4: value (none) -> PBPC
- R1, R2: value 68 -> 68R
